File: AquaTicker/aqua_ticker.kicad_pcb (KiCad board)
At the start: 2 copper layers, 99.4 x 76.5 mm, 129 parts, among them J1 M024MM-X, J2 M065MM, J3 RFTX, J4 Ethernet, J5 Zone Expander, J6 USB_B_Micro, J7 M085MM-8, J8 0.96inch OLED, Q1 Q_NPN_BCE, Q2 Q_NPN_BCE, SW1 SW_SPST, SW2 SW_SPST, SW3 SW_SPST, T1 Z0103MN5AA4, T2 Z0103MN5AA4, T3 Z0103MN5AA4, T4 Z0103MN5AA4, T5 Z0103MN5AA4, T6 Z0103MN5AA4, T7 Z0103MN5AA4, T8 Z0103MN5AA4, U1 XL1509-5.0E1, U2 LM358, U3 AMS1117-3.3V, U4 PSM712-LF-T7, U5 CP2102-GMR, U6 ESP32-WROOM-32D, U7 PCF8563T, U8 TCA9555PWR, U9 E22-900M30S-SX1262, Y1 Crystal_Small

Commit message: AquaTicker initial commit
Parts:
- SP1, SP2, SP3, SP4, SP5, SP6, SP7, SP8, SP9: footprint arilo_sprinkler:PCB-SGAP -> aqua_ticker:PCB-SGAP
Other:
- board text added: "AquaTicker Based on OpenSprinkler"
- board text removed: "AriloSprinkler 8-Zone 24VAC @Javier Arigita (OS based)"
- board text removed: "AriloSprinkler 8-Zone 24VAC @Javier Arigita OpenSprinkler based"
Changed lines of the file:
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@@
     )
   )
-  (module arilo_sprinkler:PCB-SGAP (layer Top)
+  (module aqua_ticker:PCB-SGAP (layer Top)
     (at 114.4143 114.8461 180)
     (attr smd)
@@
       (net 1 GND) (solder_mask_margin 0.0508) (solder_paste_margin -0.0508) (zone_connect 2))
   )
-  (module arilo_sprinkler:PCB-SGAP (layer Top)
+  (module aqua_ticker:PCB-SGAP (layer Top)
     (at 145.3891 115.2496 90)
     (attr smd)
@@
       (net 67 "Net-(J7-Pad1)") (solder_mask_margin 0.0508) (solder_paste_margin -0.0508) (zone_connect 2))
   )
-  (module arilo_sprinkler:PCB-SGAP (layer Top)
+  (module aqua_ticker:PCB-SGAP (layer Top)
     (at 151.1554 115.2652 90)
     (attr smd)
@@
       (net 66 "Net-(J7-Pad2)") (solder_mask_margin 0.0508) (solder_paste_margin -0.0508) (zone_connect 2))
   )
-  (module arilo_sprinkler:PCB-SGAP (layer Top)
+  (module aqua_ticker:PCB-SGAP (layer Top)
     (at 157.5481 115.2496 90)
     (attr smd)
@@
       (net 65 "Net-(J7-Pad3)") (solder_mask_margin 0.0508) (solder_paste_margin -0.0508) (zone_connect 2))
   )
-  (module arilo_sprinkler:PCB-SGAP (layer Top)
+  (module aqua_ticker:PCB-SGAP (layer Top)
     (at 164.719 115.2652 90)
     (attr smd)
@@
       (net 64 "Net-(J7-Pad4)") (solder_mask_margin 0.0508) (solder_paste_margin -0.0508) (zone_connect 2))
   )
-  (module arilo_sprinkler:PCB-SGAP (layer Top)
+  (module aqua_ticker:PCB-SGAP (layer Top)
     (at 172.085 115.2554 90)
     (attr smd)
@@
       (net 63 "Net-(J7-Pad5)") (solder_mask_margin 0.0508) (solder_paste_margin -0.0508) (zone_connect 2))
   )
-  (module arilo_sprinkler:PCB-SGAP (layer Top)
+  (module aqua_ticker:PCB-SGAP (layer Top)
     (at 186.309 115.2398 90)
     (attr smd)
@@
       (net 61 "Net-(J7-Pad7)") (solder_mask_margin 0.0508) (solder_paste_margin -0.0508) (zone_connect 2))
   )
-  (module arilo_sprinkler:PCB-SGAP (layer Top)
+  (module aqua_ticker:PCB-SGAP (layer Top)
     (at 192.4541 115.3766 90)
     (attr smd)
@@
       (net 60 "Net-(J7-Pad8)") (solder_mask_margin 0.0508) (solder_paste_margin -0.0508) (zone_connect 2))
   )
-  (module arilo_sprinkler:PCB-SGAP (layer Top)
+  (module aqua_ticker:PCB-SGAP (layer Top)
     (at 179.2986 115.23 90)
     (attr smd)
@@
     (effects (font (size 0.6 0.6) (thickness 0.115)) (justify left bottom))
   )
-  (gr_text "AriloSprinkler 8-Zone 24VAC\n@Javier Arigita\nOpenSprinkler based" (at 172.4533 105.1306) (layer B.SilkS)
+  (gr_text "AquaTicker\n\nBased on OpenSprinkler" (at 172.4533 105.1306) (layer B.SilkS)
     (effects (font (size 1.5 1.5) (thickness 0.15)) (justify mirror))
   )
@@
     (effects (font (size 0.77216 0.77216) (thickness 0.115824)) (justify bottom))
   )
-  (gr_text "AriloSprinkler 8-Zone 24VAC\n@Javier Arigita (OS based)" (at 101.0412 93.2688 90) (layer F.SilkS)
+  (gr_text "AquaTicker\n\nBased on OpenSprinkler" (at 101.0412 93.2688 90) (layer F.SilkS)
     (effects (font (size 1 1) (thickness 0.15)))
   )
